File: Shield_Brazo_V1.0/Drivers.kicad_sch (KiCad schematic)
At the start: 15 parts, among them J10 CON_M3, J11 CON_M6, J12 CON_M5, J13 CON_M4, J5 STEPS, J6 CON_M1, J7 STEPS, J8 CON_M2, J9 STEPS, U3 TMC2209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

Commit message: Laptop
Parts:
- C3, C4, C5: footprint PCM_Capacitor_THT_AKL:CP_Radial_D8.0mm_P3.80mm -> PCM_Capacitor_THT_AKL:CP_Radial_D6.3mm_P2.50mm
Changed lines of the file:
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@@
 			)
 		)
-		(property "Footprint" "PCM_Capacitor_THT_AKL:CP_Radial_D8.0mm_P3.80mm"
+		(property "Footprint" "PCM_Capacitor_THT_AKL:CP_Radial_D6.3mm_P2.50mm"
 			(at 87.63 109.22 0)
 			(effects
@@
 			)
 		)
-		(property "Footprint" "PCM_Capacitor_THT_AKL:CP_Radial_D8.0mm_P3.80mm"
+		(property "Footprint" "PCM_Capacitor_THT_AKL:CP_Radial_D6.3mm_P2.50mm"
 			(at 97.79 36.83 0)
 			(effects
@@
 			)
 		)
-		(property "Footprint" "PCM_Capacitor_THT_AKL:CP_Radial_D8.0mm_P3.80mm"
+		(property "Footprint" "PCM_Capacitor_THT_AKL:CP_Radial_D6.3mm_P2.50mm"
 			(at 187.96 109.22 0)
 			(effects
