File: Shield_Brazo_V1.0/Shield_Brazo_V1.0.kicad_pcb (KiCad board)
At the start: 2 copper layers, 95 x 132.5 mm, 48 parts, among them J10 CON_M3, J11 CON_M6, J12 CON_M5, J13 CON_M4, J14 VIN_M6-M2, J2 Barrel_Jack_Switch, J3 I2C, J4 UART, J5 STEPS, J6 CON_M1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

Commit message: Laptop
Parts:
- removed D1: LED_V1, PCM_LED_THT_AKL:LED_D5.0mm
- removed R1: 2K 1W, Resistor_THT:R_Axial_DIN0207_L6.3mm_D2.5mm_P15.24mm_Horizontal
- added C7: 100uF/25V, PCM_Capacitor_THT_AKL:CP_Radial_D16.0mm_P7.50mm, F.Cu at (79.1, 70.5)
- C3, C4, C5: footprint PCM_Capacitor_THT_AKL:CP_Radial_D8.0mm_P3.80mm -> PCM_Capacitor_THT_AKL:CP_Radial_D6.3mm_P2.50mm
- moved J14 1.27 mm to (73.0, 56.5)
Routing:
- net Net-(D1-A): track 6.51 -> 0.00 mm
- net +12V_M6M2: track 113.8 -> 119.2 mm
- net GND: track 86.8 -> 88.4 mm
- net /Drivers/DIR_M3: track 106.9 -> 108.3 mm
- net /Drivers/STEP_M3: track 108.0 -> 109.3 mm
- net /Drivers/STEP_M2: track 86.3 -> 87.4 mm
- net /Drivers/STEP_M1: track 71.5 -> 72.2 mm
- net /MCU/TX: track 37.0 -> 37.1 mm, vias 1 -> 2
