File: Shield_Brazo_V1.0/Shield_Brazo_V1.0.kicad_sch (KiCad schematic)
At the start: 0 parts

Commit message: Terminada, Revision
Other:
- added sheet Drivers (Drivers.kicad_sch)
- added sheet MCU (MCU.kicad_sch)
- added sheet Outputs (untitled.kicad_sch)
- added sheet Pinout (Pinout.kicad_sch)
- added sheet Power (Power.kicad_sch)
